File: Hardware/InkTime_v2.brd (EAGLE design)
At the start: 46 x 35 mm, 105 parts, among them IC1 BQ25180YBGR_BQ25180YBGR, IC2 DRV2605YZFR, IC3 BMA423, IC9 RT6160AWSC, J1 503480-2400, J2 TC2030-IDC, J4 KH-TYPE-C-16P, Q1 20V/4.2A/52mΩ/1.4W, Q3 SI1308EDL-T1-GE3, U1 NRF52840_QF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

Commit message: fix review issues
Signed-off-by: Cristi <cristimacovei26@gmail.com>
Routing:
- net D-: track 12.4 -> 15.9 mm
- net RESE: track 21.6 -> 21.1 mm
